Commit message: URDF adjusted for simulation

File: urdf/four_dof_manipulator.urdf (robot description, URDF)
Before this commit: robot four_dof_manipulator, 5 links, 4 joints
Links:
- added link world
Joints:
- added joint fixed: type fixed, parent world, child base_link
- joint joint_1: limit lower=-1.5708 upper=1.5708 effort=0 velocity=2 -> lower=-1.5708 upper=1.5708 effort=500 velocity=2; origin xyz=-0.002088 -0.2 -0.0041908 rpy=-3.1416 0 0.011071 -> xyz=-0.002088 -0.2 -0.0041908 rpy=-3.1416 0 -3.1416
- joint joint_2: limit lower=-2.0944 upper=0.5236 effort=0 velocity=2 -> lower=-1.2217304764 upper=1.9198621772 effort=500 velocity=2
- joint joint_3: limit lower=-3.8397 upper=-2.0944 effort=0 velocity=2 -> lower=-1.9198621772 upper=-6.6322511576 effort=500 velocity=2
- joint joint_4: limit lower=0.34907 upper=1.0472 effort=0 velocity=2 -> lower=0.6981317008 upper=-2.4434609528 effort=500 velocity=2

Commit message: joint limits adjusted

File: urdf/four_dof_manipulator.urdf (robot description, URDF)
Before this commit: robot four_dof_manipulator, 6 links, 5 joints
Joints:
- joint joint_3: limit lower=-1.9198621772 upper=-6.6322511576 effort=500 velocity=2 -> lower=-6.6322511576 upper=-1.9198621772 effort=500 velocity=2
- joint joint_4: limit lower=0.6981317008 upper=-2.4434609528 effort=500 velocity=2 -> lower=-2.4434609528 upper=0.6981317008 effort=500 velocity=2

Commit message: 3rd joint range config

File: urdf/four_dof_manipulator.urdf (robot description, URDF)
Before this commit: robot four_dof_manipulator, 6 links, 5 joints
Joints:
- joint joint_1: limit lower=-1.5708 upper=1.5708 effort=500 velocity=2 -> lower=-1.5707963268 upper=1.5707963268 effort=500 velocity=2
- joint joint_3: limit lower=-6.6322511576 upper=-1.9198621772 effort=500 velocity=2 -> lower=-6.2831853072 upper=-2.2689280276 effort=500 velocity=2

Commit message: gazebo simulation environment configs

File: urdf/four_dof_manipulator.urdf (robot description, URDF)
Before this commit: robot four_dof_manipulator, 6 links, 5 joints
Joints:
- joint fixed: origin (none) -> xyz=0.0 0.0 0.068 rpy=0.0 0.0 0.0

Commit message: similation environment

File: urdf/four_dof_manipulator.urdf (robot description, URDF)
Before this commit: robot four_dof_manipulator, 6 links, 5 joints
Links:
- added link table; visual box size=0.6 0.4 0.9
Joints:
- added joint table_joint: type fixed, parent table, child base_link, origin xyz=0.0 0.0 0.518 rpy=0.0 0.0 0.0
- joint fixed: child base_link -> table; origin xyz=0.0 0.0 0.068 rpy=0.0 0.0 0.0 -> xyz=0.0 0.0 0.450 rpy=0.0 0.0 0.0

Commit message: end effector settings

File: urdf/four_dof_manipulator.urdf (robot description, URDF)
Before this commit: robot four_dof_manipulator, 7 links, 6 joints
Links:
- removed link last_link
- added link finger_1, mass 0.00371707887588344; collision mesh filename=package://four_dof_manipulator/meshes/finger_1.STL; visual mesh filename=package://four_dof_manipulator/meshes/finger_1.STL
- added link finger_2, mass 0.00354537803339804; collision mesh filename=package://four_dof_manipulator/meshes/finger_2.STL; visual mesh filename=package://four_dof_manipulator/meshes/finger_2.STL
- added link fourth_link, mass 0.114529356723246; collision mesh filename=package://four_dof_manipulator/meshes/fourth_link.STL; visual mesh filename=package://four_dof_manipulator/meshes/fourth_link.STL
Joints:
- added joint finger1: type revolute, parent fourth_link, child finger_1, origin xyz=-0.0425 -0.006 0.092879 rpy=-1.4841 0 1.5708, axis 1 0 0, limit lower=-0.3 upper=0.3 effort=500 velocity=2
- added joint finger2: type revolute, parent fourth_link, child finger_2, origin xyz=-0.0695 -0.006 0.092879 rpy=1.5656 0 1.5708, axis 1 0 0, limit lower=0 upper=0.6 effort=500 velocity=2
- joint joint_1: origin xyz=-0.002088 -0.2 -0.0041908 rpy=-3.1416 0 -3.1416 -> xyz=-0.00208795693759905 -0.199999999999975 -0.00419080295344085 rpy=-3.14159265358979 0 0.0110713534620342
- joint joint_2: origin xyz=0 -0.068 -0.117 rpy=-1.5708 1.231 0 -> xyz=0 -0.0680000000000001 -0.117000000000003 rpy=-1.5707963267949 1.23097997933017 0
- joint joint_4: child last_link -> fourth_link

Commit message: end effector config

File: urdf/four_dof_manipulator.urdf (robot description, URDF)
Before this commit: robot four_dof_manipulator, 9 links, 8 joints
Links:
- link finger_1: mass 0.00371707887588344 -> 0.00517538664215202
- link finger_2: mass 0.00354537803339804 -> 0.0050037
Joints:
- joint finger2: limit lower=0 upper=0.6 effort=500 velocity=2 -> lower=-0.3 upper=0.3 effort=500 velocity=2
